Commit message: analysis

File: src/ethercat_ROS2/src/zeroerr_driver_ros2/description/ros2_control/motor_drive.ros2_control.xacro (robot description, xacro)
@@ -12,11 +12,21 @@
         <state_interface name="position"/>
         <state_interface name="velocity"/>
+        <state_interface name="bus_voltage"/>
         <command_interface name="position"/>
         <command_interface name="velocity"/>
-        <ec_module name="ZeroErr_joint_1">
+        <state_interface name="current"/>
+        <state_interface name="velocity_demand"/>
+        <state_interface name="torque_demand"/>
+        <state_interface name="position_demand"/>
+        <state_interface name="touch_probe_status"/>
+        <state_interface name="digital_inputs"/>
+        <state_interface name="status_word"/>
+        <state_interface name="mode_of_operation"/>
+        <state_interface name="error_code"/>
+          <ec_module name="ZeroErr_joint_1">
           <plugin>ethercat_generic_plugins/EcCiA402Drive</plugin>
           <param name="alias">0</param>
           <param name="position">0</param>
-          <param name="mode_of_operation">8</param>
+          <param name="mode_of_operation">9</param>
           <param name="slave_config">$(find ethercat_zeroerr)/config/zeroerr_config.yaml</param>
         </ec_module>
@@ -25,11 +35,21 @@
         <state_interface name="position"/>
         <state_interface name="velocity"/>
+        <state_interface name="bus_voltage"/>
         <command_interface name="position"/>
         <command_interface name="velocity"/>
-        <ec_module name="ZeroErr_joint_2">
+        <state_interface name="current"/>
+        <state_interface name="velocity_demand"/>
+        <state_interface name="torque_demand"/>
+        <state_interface name="position_demand"/>
+        <state_interface name="touch_probe_status"/>
+        <state_interface name="digital_inputs"/>
+        <state_interface name="status_word"/>
+        <state_interface name="mode_of_operation"/>
+        <state_interface name="error_code"/>
+          <ec_module name="ZeroErr_joint_2">
           <plugin>ethercat_generic_plugins/EcCiA402Drive</plugin>
           <param name="alias">0</param>
           <param name="position">1</param>
-          <param name="mode_of_operation">8</param>
+          <param name="mode_of_operation">9</param>
           <param name="slave_config">$(find ethercat_zeroerr)/config/zeroerr_config.yaml</param>
         </ec_module>
@@ -38,11 +58,21 @@
         <state_interface name="position"/>
         <state_interface name="velocity"/>
+        <state_interface name="bus_voltage"/>
         <command_interface name="position"/>
         <command_interface name="velocity"/>
+        <state_interface name="current"/>
+        <state_interface name="velocity_demand"/>
+        <state_interface name="torque_demand"/>
+        <state_interface name="position_demand"/>
+        <state_interface name="touch_probe_status"/>
+        <state_interface name="digital_inputs"/>
+        <state_interface name="status_word"/>
+        <state_interface name="mode_of_operation"/>
+        <state_interface name="error_code"/>
         <ec_module name="ZeroErr_joint_3">
           <plugin>ethercat_generic_plugins/EcCiA402Drive</plugin>
           <param name="alias">0</param>
           <param name="position">2</param>
-          <param name="mode_of_operation">8</param>
+          <param name="mode_of_operation">9</param>
           <param name="slave_config">$(find ethercat_zeroerr)/config/zeroerr_config.yaml</param>
         </ec_module>
@@ -51,11 +81,21 @@
         <state_interface name="position"/>
         <state_interface name="velocity"/>
+        <state_interface name="bus_voltage"/>
         <command_interface name="position"/>
         <command_interface name="velocity"/>
+        <state_interface name="current"/>
+        <state_interface name="velocity_demand"/>
+        <state_interface name="torque_demand"/>
+        <state_interface name="position_demand"/>
+        <state_interface name="touch_probe_status"/>
+        <state_interface name="digital_inputs"/>
+        <state_interface name="status_word"/>
+        <state_interface name="mode_of_operation"/>
+        <state_interface name="error_code"/>
         <ec_module name="ZeroErr_joint_4">
           <plugin>ethercat_generic_plugins/EcCiA402Drive</plugin>
           <param name="alias">0</param>
           <param name="position">3</param>
-          <param name="mode_of_operation">8</param>
+          <param name="mode_of_operation">9</param>
           <param name="slave_config">$(find ethercat_zeroerr)/config/zeroerr_config.yaml</param>
         </ec_module>
@@ -64,11 +104,21 @@
         <state_interface name="position"/>
         <state_interface name="velocity"/>
+        <state_interface name="bus_voltage"/>
         <command_interface name="position"/>
         <command_interface name="velocity"/>
+        <state_interface name="current"/>
+        <state_interface name="velocity_demand"/>
+        <state_interface name="torque_demand"/>
+        <state_interface name="position_demand"/>
+        <state_interface name="touch_probe_status"/>
+        <state_interface name="digital_inputs"/>
+        <state_interface name="status_word"/>
+        <state_interface name="mode_of_operation"/>
+        <state_interface name="error_code"/>
         <ec_module name="ZeroErr_joint_5">
           <plugin>ethercat_generic_plugins/EcCiA402Drive</plugin>
           <param name="alias">0</param>
           <param name="position">4</param>
-          <param name="mode_of_operation">8</param>
+          <param name="mode_of_operation">9</param>
           <param name="slave_config">$(find ethercat_zeroerr)/config/zeroerr_config.yaml</param>
         </ec_module>

File: src/plex_arm_urdf_3/urdf/plex_arm_urdf_3.urdf.xacro (robot description, xacro)
@@ -18,6 +18,6 @@
   <xacro:property name="color_blue"         value="0.86667 0.9098  1       1" />
   <!-- Placeholder limits — fill these in per-joint once confirmed -->
-  <xacro:property name="default_effort"     value="0" />
-  <xacro:property name="default_velocity"   value="0" />
+  <xacro:property name="default_effort"     value="100" />
+  <xacro:property name="default_velocity"   value="100" />
   <!-- ============================================================
        Macros
