Commit message: ARM WORKS

File: src/plex_arm_urdf_3/urdf/plex_arm_urdf_3.urdf.xacro (robot description, xacro)
@@ -1,10 +1,29 @@
 <?xml version="1.0" encoding="utf-8"?>
-<robot name="plex_arm_urdf_3" xmlns:xacro="http://www.ros.org/wiki/xacro">
-  <!-- ===================== PROPERTIES ===================== -->
-  <!-- Colors -->
-  <xacro:property name="color_grey"  value="0.75294 0.75294 0.75294 1" />
-  <xacro:property name="color_blue"  value="0.86667 0.9098 1 1" />
-  <!-- ===================== MACROS ===================== -->
-  <xacro:macro name="default_inertial" params="mass ixx ixy ixz iyy iyz izz ox oy oz">
+<!--
+  plex_arm_2_v2.urdf.xacro
+  Xacro conversion of SolidWorks-exported URDF for plex_arm_2 (re-export).
+  Originally generated by sw_urdf_exporter (Stephen Brawner).
+  Usage:
+    xacro plex_arm_2_v2.urdf.xacro > plex_arm_2_v2.urdf
+    check_urdf plex_arm_2_v2.urdf
+  NOTE: All joint limits are currently 0/0 as exported from SolidWorks.
+        Update lower/upper/effort/velocity before using with MoveIt or hardware.
+-->
+<robot name="plex_arm_2" xmlns:xacro="http://www.ros.org/wiki/xacro">
+  <!-- ============================================================
+       Properties
+       ============================================================ -->
+  <xacro:property name="mesh_pkg"           value="plex_arm_2" />
+  <xacro:property name="color_grey"         value="0.75294 0.75294 0.75294 1" />
+  <xacro:property name="color_blue"         value="0.86667 0.9098  1       1" />
+  <!-- Placeholder limits — fill these in per-joint once confirmed -->
+  <xacro:property name="default_effort"     value="0" />
+  <xacro:property name="default_velocity"   value="0" />
+  <!-- ============================================================
+       Macros
+       ============================================================ -->
+  <!-- Inertial block -->
+  <xacro:macro name="inertial"
+               params="ox oy oz mass ixx ixy ixz iyy iyz izz">
     <inertial>
       <origin xyz="${ox} ${oy} ${oz}" rpy="0 0 0" />
@@ -14,89 +33,127 @@
     </inertial>
   </xacro:macro>
-  <xacro:macro name="mesh_link" params="name color mesh_file ox oy oz
-               mass ixx ixy ixz iyy iyz izz">
-    <link name="${name}">
-      <xacro:default_inertial mass="${mass}"
-        ixx="${ixx}" ixy="${ixy}" ixz="${ixz}"
-        iyy="${iyy}" iyz="${iyz}" izz="${izz}"
-        ox="${ox}" oy="${oy}" oz="${oz}" />
-      <visual>
-        <origin xyz="0 0 0" rpy="0 0 0" />
-        <geometry>
-          <mesh filename="package://plex_arm_urdf_3/meshes/${mesh_file}.STL" />
-        </geometry>
-        <material name="">
-          <color rgba="${color}" />
-        </material>
-      </visual>
-      <collision>
-        <origin xyz="0 0 0" rpy="0 0 0" />
-        <geometry>
-          <mesh filename="package://plex_arm_urdf_3/meshes/${mesh_file}.STL" />
-        </geometry>
-      </collision>
-    </link>
+  <!-- Visual + collision (mesh-based) -->
+  <xacro:macro name="mesh_geometry"
+               params="link_name color_rgba">
+    <visual>
+      <origin xyz="0 0 0" rpy="0 0 0" />
+      <geometry>
+        <mesh filename="package://${mesh_pkg}/meshes/${link_name}.STL" />
+      </geometry>
+      <material name="">
+        <color rgba="${color_rgba}" />
+      </material>
+    </visual>
+    <collision>
+      <origin xyz="0 0 0" rpy="0 0 0" />
+      <geometry>
+        <mesh filename="package://${mesh_pkg}/meshes/${link_name}.STL" />
+      </geometry>
+    </collision>
   </xacro:macro>
-  <!-- ===================== LINKS ===================== -->
-  <xacro:mesh_link name="base_link" color="${color_grey}" mesh_file="base_link"
-    ox="-2.2467E-05" oy="-1.5826E-05" oz="0.037461"
-    mass="0.39916"
-    ixx="0.00032485" ixy="5.025E-08"  ixz="-2.2819E-07"
-    iyy="0.00032522" iyz="-1.8676E-07" izz="0.00048667" />
-  <xacro:mesh_link name="link_2" color="${color_blue}" mesh_file="link_2"
-    ox="0.0021138" oy="-0.016329" oz="0.052462"
-    mass="1.0133"
-    ixx="0.0014335" ixy="-1.4203E-05" ixz="7.5921E-06"
-    iyy="0.001499"  iyz="0.00012324"  izz="0.0014189" />
-  <xacro:mesh_link name="link_3" color="${color_grey}" mesh_file="link_3"
-    ox="0.26754" oy="0.053738" oz="-0.031859"
-    mass="1.3505"
-    ixx="0.0013405" ixy="4.1403E-05" ixz="0.0002258"
-    iyy="0.0032102" iyz="-5.27E-06"  izz="0.0031982" />
-  <xacro:mesh_link name="link_4" color="${color_grey}" mesh_file="link_4"
-    ox="0.082946" oy="-0.041589" oz="0.059096"
-    mass="0.53981"
-    ixx="0.0004222"  ixy="7.614E-06"  ixz="-0.00010509"
-    iyy="0.00066838" iyz="6.346E-06"  izz="0.00062584" />
-  <xacro:mesh_link name="link_5" color="${color_grey}" mesh_file="link_5"
-    ox="0.015109" oy="-0.00066097" oz="0.23769"
-    mass="0.56411"
-    ixx="0.0011559" ixy="1.6719E-06"  ixz="-5.4768E-05"
-    iyy="0.0011686" iyz="7.9723E-07"  izz="0.00028936" />
-  <xacro:mesh_link name="link_6" color="${color_grey}" mesh_file="link_6"
-    ox="0.037346" oy="-0.016629" oz="0.039697"
-    mass="0.20707"
-    ixx="8.7908E-05"  ixy="1.4913E-05"  ixz="2.6473E-05"
-    iyy="0.00015558"  iyz="-6.0339E-06" izz="0.00012787" />
-  <!-- ===================== JOINTS ===================== -->
-  <joint name="joint_1" type="continuous">
-    <origin xyz="0 0 0.0641" rpy="0 0 0" />
+  <!-- ============================================================
+       Links
+       ============================================================ -->
+  <!-- Base turntable / mounting plate -->
+  <link name="base_link">
+    <xacro:inertial
+      ox="0.0013285"  oy="-0.0013224" oz="0.037461"
+      mass="0.39916"
+      ixx="0.00032485" ixy="5.025E-08"   ixz="-2.2819E-07"
+      iyy="0.00032522" iyz="-1.8676E-07" izz="0.00048667" />
+    <xacro:mesh_geometry link_name="base_link" color_rgba="${color_grey}" />
+  </link>
+  <!-- Shoulder / first rotating link -->
+  <link name="link_2">
+    <xacro:inertial
+      ox="6.3613E-05"  oy="-0.016265" oz="0.055354"
+      mass="1.0133"
+      ixx="0.0014695" ixy="-6.0098E-08" ixz="5.8462E-08"
+      iyy="0.0014982" iyz="0.00010509"  izz="0.0013838" />
+    <xacro:mesh_geometry link_name="link_2" color_rgba="${color_blue}" />
+  </link>
+  <!-- Upper arm -->
+  <link name="link_3">
+    <xacro:inertial
+      ox="0.00048454" oy="0.0020711" oz="-0.10143"
+      mass="1.3505"
+      ixx="0.0032252" ixy="3.0835E-07"  ixz="9.0245E-06"
+      iyy="0.003211"  iyz="-1.0066E-05" izz="0.0013126" />
+    <xacro:mesh_geometry link_name="link_3" color_rgba="${color_grey}" />
+  </link>
+  <!-- Forearm -->
+  <link name="link_4">
+    <xacro:inertial
+      ox="-0.010201" oy="0.01352" oz="0.028625"
+      mass="0.53981"
+      ixx="0.00043641" ixy="6.5099E-07"  ixz="-0.00011755"
+      iyy="0.00066866" iyz="3.5023E-06"  izz="0.00061134" />
+    <xacro:mesh_geometry link_name="link_4" color_rgba="${color_grey}" />
+  </link>
+  <!-- Wrist pitch -->
+  <link name="link_5">
+    <xacro:inertial
+      ox="-5.2719E-06" oy="0.0036972" oz="-0.068702"
+      mass="0.56411"
+      ixx="0.0011591" ixy="-2.4169E-07" ixz="3.1175E-07"
+      iyy="0.0011689" iyz="4.9596E-07"  izz="0.00028591" />
+    <xacro:mesh_geometry link_name="link_5" color_rgba="${color_grey}" />
+  </link>
+  <!-- End-effector / wrist roll -->
+  <link name="link_6">
+    <xacro:inertial
+      ox="-0.028222" oy="-0.0034544" oz="-0.0084206"
+      mass="0.20707"
+      ixx="7.2186E-05"  ixy="7.9371E-07" ixz="-5.9922E-06"
+      iyy="0.00015872"  iyz="5.479E-08"  izz="0.00014045" />
+    <xacro:mesh_geometry link_name="link_6" color_rgba="${color_grey}" />
+  </link>
+  <!-- ============================================================
+       Joints
+       ============================================================ -->
+  <!-- joint_1 : base_link → link_2  (shoulder yaw, ~Z axis) -->
+  <joint name="joint_1" type="revolute">
+    <origin xyz="0.0013509 -0.0013066 0.0641" rpy="0 -0.0012835 -0.027488" />
     <parent link="base_link" />
     <child  link="link_2" />
-    <axis   xyz="0 0 1" />
+    <axis   xyz="0.0012835 0 1" />
+    <limit lower="-3.14" upper="3.14"
+           effort="${default_effort}" velocity="${default_velocity}" />
   </joint>
-  <joint name="joint_2" type="continuous">
-    <origin xyz="-0.0016216 -0.058978 0.063" rpy="0 0 0" />
+  <!-- joint_2 : link_2 → link_3  (upper-arm pitch, −Y axis) -->
+  <joint name="joint_2" type="revolute">
+    <origin xyz="-0.0011924 0 0.4323" rpy="0 0.0012835 0" />
     <parent link="link_2" />
     <child  link="link_3" />
-    <axis   xyz="-0.027485 -0.99962 0" />
+    <axis   xyz="0 -1 0" />
+    <limit lower="-3.14" upper="3.14"
+           effort="${default_effort}" velocity="${default_velocity}" />
   </joint>
-  <joint name="joint_3" type="continuous">
-    <origin xyz="0.42375 0.10171 -0.050398" rpy="0 0 0" />
+  <!-- joint_3 : link_3 → link_4  (elbow pitch, −Y axis) -->
+  <joint name="joint_3" type="revolute">
+    <origin xyz="0.089987 0.0015 0.090304" rpy="0 0 0" />
     <parent link="link_3" />
     <child  link="link_4" />
-    <axis   xyz="-0.027485 -0.99962 0" />
+    <axis   xyz="0 -1 0" />
+    <limit lower="-3.14" upper="3.14"
+           effort="${default_effort}" velocity="${default_velocity}" />
   </joint>
-  <joint name="joint_4" type="continuous">
-    <origin xyz="0.096215 -0.055479 0.11335" rpy="0 0 0" />
+  <!-- joint_4 : link_4 → link_5  (wrist pitch, ~Z axis) -->
+  <joint name="joint_4" type="revolute">
+    <origin xyz="-0.00041051 -0.0034488 0.39053" rpy="0 0 0" />
     <parent link="link_4" />
     <child  link="link_5" />
-    <axis   xyz="0.063628 -0.0017495 0.99797" />
+    <axis   xyz="-0.0012835 0 1" />
+    <limit lower="-3.14" upper="3.14"
+           effort="${default_effort}" velocity="${default_velocity}" />
   </joint>
-  <joint name="joint_5" type="continuous">
-    <origin xyz="0.019526 -0.00053686 0.30625" rpy="0 0 0" />
+  <!-- joint_5 : link_5 → link_6  (wrist roll, ~Y axis) -->
+  <joint name="joint_5" type="revolute">
+    <origin xyz="0.0049507 0.016857 0.059516" rpy="0 0 0" />
     <parent link="link_5" />
     <child  link="link_6" />
-    <axis   xyz="-0.16576 -0.98613 0.00884" />
+    <axis   xyz="-0.026297 0.99965 -3.3751E-05" />
+    <limit lower="-3.14" upper="3.14"
+           effort="${default_effort}" velocity="${default_velocity}" />
   </joint>
 </robot>
