Commit message: replaced redundant plex_arm_2 with updated plex_arm_3

File: src/plex_arm_urdf_3/urdf/plex_arm_urdf_3.urdf.xacro (robot description, xacro)
@@ -114,5 +114,5 @@
   <!-- joint_1 : base_link → link_2  (shoulder yaw, ~Z axis) -->
   <joint name="joint_1" type="revolute">
-    <origin xyz="0.0013509 -0.0013066 0.0641" rpy="0 -0.0012835 -0.027488" />
+    <origin xyz="0.0013509 -0.0013066 0.0641" rpy="0 -0.0012835 -0.027488"/>
     <parent link="base_link" />
     <child  link="link_2" />
@@ -123,5 +123,5 @@
   <!-- joint_2 : link_2 → link_3  (upper-arm pitch, −Y axis) -->
   <joint name="joint_2" type="revolute">
-    <origin xyz="-0.0011924 0 0.4323" rpy="0 0.0012835 0" />
+    <origin xyz="-0.0011924 0 0.4323" rpy="0 0 0" />
     <parent link="link_2" />
     <child  link="link_3" />
